File: Hardware/Proto_Pedal.sch (EAGLE design)
At the start: 124 parts, among them Q1 2.5A/30V

Commit message: Fixing what Eric found in review.
-I/O coupling caps now have similar trace arrangements.
-Second page of Schem bumped to V10.
Other:
- note removed: "V02"
Changed lines of the file:
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@@
 <plain>
 <text x="167.64" y="7.62" size="2.54" layer="94" font="vector">Byron Jacquot</text>
-<text x="238.76" y="7.62" size="2.54" layer="94" font="vector">V02</text>
+<text x="238.76" y="7.62" size="2.54" layer="94" font="vector">V10</text>
 <text x="91.44" y="5.08" size="3.81" layer="97">30-row DIP proto area</text>
 </plain>
